Commit message: fix absolute paths and cmake

File: model/panda/panda.urdf (robot description, URDF)
Before this commit: robot panda, 10 links, 9 joints
Links:
- link leftfinger: geometry visual mesh filename=meshes/visual/finger.obj
- link link0: geometry visual mesh filename=meshes/visual/link0.obj
- link link1: geometry visual mesh filename=meshes/visual/link1.obj
- link link2: geometry visual mesh filename=meshes/visual/link2.obj
- link link3: geometry visual mesh filename=meshes/visual/link3.obj
- link link4: geometry visual mesh filename=meshes/visual/link4.obj
- link link5: geometry visual mesh filename=meshes/visual/link5.obj
- link link6: geometry visual mesh filename=meshes/visual/link6.obj
- link link7: geometry visual mesh filename=meshes/visual/hand.obj; visual mesh filename=meshes/visual/link7.obj
- link rightfinger: geometry visual mesh filename=meshes/visual/finger.obj

Commit message: enable robot collision

File: model/panda/panda.urdf (robot description, URDF)
Before this commit: robot panda, 10 links, 9 joints
Links:
- link leftfinger: geometry collision mesh filename=meshes/collision/finger.obj; visual mesh filename=meshes/visual/finger.obj
- link link0: geometry collision mesh filename=meshes/collision/link0.obj; visual mesh filename=meshes/visual/link0.obj
- link link1: geometry collision mesh filename=meshes/collision/link1.obj; visual mesh filename=meshes/visual/link1.obj
- link link2: geometry collision mesh filename=meshes/collision/link2.obj; visual mesh filename=meshes/visual/link2.obj
- link link3: geometry collision mesh filename=meshes/collision/link3.obj; visual mesh filename=meshes/visual/link3.obj
- link link4: geometry collision mesh filename=meshes/collision/link4.obj; visual mesh filename=meshes/visual/link4.obj
- link link5: geometry collision mesh filename=meshes/collision/link5.obj; visual mesh filename=meshes/visual/link5.obj
- link link6: geometry collision mesh filename=meshes/collision/link6.obj; visual mesh filename=meshes/visual/link6.obj
- link link7: geometry collision mesh filename=meshes/collision/hand.obj; collision mesh filename=meshes/collision/link7.obj
- link rightfinger: geometry collision mesh filename=meshes/collision/finger.obj; visual mesh filename=meshes/visual/finger.obj

Commit message: make figer collision basic boxes instead of mesh

File: model/panda/panda.urdf (robot description, URDF)
Before this commit: robot panda, 10 links, 9 joints
Links:
- link leftfinger: geometry collision box size=0.015 0.01 0.045; visual mesh filename=meshes/visual/finger.obj
- link rightfinger: geometry collision box size=0.015 0.01 0.045; visual mesh filename=meshes/visual/finger.obj

Commit message: example motion with visual sphere at ee

File: model/panda/panda.urdf (robot description, URDF)
Before this commit: robot panda, 10 links, 9 joints
Links:
- link link7: geometry collision mesh filename=meshes/collision/hand.obj; collision mesh filename=meshes/collision/link7.obj
